File: dingoPDM-Max/BTS700n_1EPP.kicad_sch (KiCad schematic)
At the start: 13 parts, among them U8 BTS70015-1ESP

Commit message: Updated to Kicad 8
Parts:
- U8: value BTS70015-1ESP -> BTS70012-1ESP

Commit message: First version ordered
Parts:
- U8: Digi-Key_PN (none) -> 448-BTS700121ESPXUMA2CT-ND
Changed lines of the file:
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@@
 	(title_block
 		(title "dingoPDM-Max")
-		(date "2024-07-06")
-		(rev "v0.1")
+		(date "2024-09-06")
+		(rev "v1.0")
 		(comment 3 "github.com/corygrant")
 		(comment 4 "Cory Grant")
@@
 			(at 132.08 104.14 0)
 			(effects
+				(font
+					(size 1.27 1.27)
+				)
+				(hide yes)
+			)
+		)
+		(property "Digi-Key_PN" "448-BTS700121ESPXUMA2CT-ND"
+			(at 132.08 104.14 0)
+			(effects

Commit message: fixed bad zone, shifted traces, increase trace widths
update part numbers for ibom
Parts:
- U8: LCSC (none) -> C3232444
Changed lines of the file:
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@@
 	(title_block
 		(title "dingoPDM-Max")
-		(date "2025-06-16")
-		(rev "v1.1")
+		(date "2025-09-29")
+		(rev "v1.2")
 		(comment 3 "github.com/corygrant")
 		(comment 4 "Cory Grant")
@@
 			(at 132.08 104.14 0)
 			(effects
+				(font
+					(size 1.27 1.27)
+				)
+				(hide yes)
+			)
+		)
+		(property "LCSC" "C3232444"
+			(at 132.08 104.14 0)
+			(effects
