File: dingoPDM-Max/HighCurrentDrivers.kicad_sch (KiCad schematic)
At the start: 6 parts, among them U7 LM324

Commit message: Updated to Kicad 8
Parts:
- renumbered C41 to C22, R8 to R17, R8 to R18, R8 to R19, R8 to R20
