File: dingoPDM-Max/Power.kicad_sch (KiCad schematic)
At the start: 18 parts, among them U1 VXO780x-500-M, U12 OKI-78SR-5_1.5-W36H-C, U13 TSR_1-2450, U2 LD1117S33CTR

Commit message: fix tvs jlc pn, #25
Parts:
- D2: LCSC C2760132 -> C152086
Changed lines of the file:
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@@
 			)
 		)
-		(property "LCSC" "C2760132"
+		(property "LCSC" "C152086"
 			(at 35.56 38.1 0)
 			(hide yes)
